Commit message: first decently working version

File: urdf/coke_can.urdf (robot description, URDF)
Before this commit: robot gripper, 1 links, 1 joints
Links:
- removed link world
- added link coke_can, mass 0.390; collision mesh filename=package://parallel_2f_gripper/meshes/coke_can.dae; visual mesh filename=package://parallel_2f_gripper/meshes/coke_can.dae
Joints:
- removed joint world_joint

File: urdf/finger.xacro (robot description, xacro)
@@ -39,5 +39,5 @@
       <child link="${prefix}crank" />
       <axis xyz="0 1 0" />
-      <limit lower="${-asin(0.5*base_x/crank_length)}" upper="${1}" velocity="5.0" effort="50" />
+      <limit lower="${-asin(0.5*base_x/crank_length)}" upper="${1}" velocity="5.0" effort="5" />
       <xacro:unless value="${mimic_joint == ''}">
         <mimic joint="${mimic_joint}" multiplier="1" offset="0" />
@@ -50,44 +50,45 @@
       <axis xyz="0 1 0" />
     </joint>
-      <joint name="${prefix}joint_1_2" type="revolute">
-        <origin xyz="0 0 ${crank_length}" rpy="0 ${pi/2} 0"/>
-        <parent link="${prefix}crank" />
-        <child link="${prefix}rod" />
-        <axis xyz="0 1 0" />
-        <limit lower="${-pi}" upper="${pi}" velocity="2.0" effort="10" />
-        <mimic joint="${prefix}finger_joint" multiplier="-1" offset="0" />
+    <joint name="${prefix}joint_1_2" type="revolute">
+      <origin xyz="0 0 ${crank_length}" rpy="0 ${pi/2} 0"/>
+      <parent link="${prefix}crank" />
+      <child link="${prefix}rod" />
+      <axis xyz="0 1 0" />
+      <limit lower="${-pi}" upper="${pi}" velocity="2.0" effort="10" />
+      <mimic joint="${prefix}finger_joint" multiplier="-1" offset="0" />
+    </joint>
+    <joint name="${prefix}joint_2_3" type="revolute">
+      <origin xyz="0 0 ${rod_length}" rpy="0 ${pi/2} 0"/>
+      <parent link="${prefix}rod" />
+      <child link="${prefix}external_crank" />
+      <axis xyz="0 1 0" />
+      <limit lower="${-pi}" upper="${pi}" velocity="2.0" effort="10" />
+      <mimic joint="${prefix}finger_joint" multiplier="1" offset="0" />
+    </joint>
+    <joint name="${prefix}joint_3_4" type="revolute">
+      <origin xyz="0 0 ${crank_length}" rpy="0 ${pi/2} 0"/>
+      <parent link="${prefix}external_crank" />
+      <child link="${prefix}base_rod" />
+      <axis xyz="0 1 0" />
+      <limit lower="${-pi}" upper="${pi}" velocity="2.0" effort="10" />
+      <mimic joint="${prefix}finger_joint" multiplier="-1" offset="0" />
+    </joint>
+    <!-- Add if to include this link only for rviz  -->
+    <!-- <link name="${prefix}tip"/>
+    <joint name="${prefix}tip_joint" type="fixed">
+      <origin xyz="${-0.5*link_width} 0 ${phalanx_length}" rpy="0 0 0"/>
+      <parent link="${prefix}phalanx" />
+      <child link="${prefix}tip" />
+    </joint> -->
+    <!-- <gazebo>
+      <joint name="${prefix}joint_4_1" type="revolute">
+        <parent>${prefix}base_rod</parent>
+        <child>${prefix}crank</child>
+        <pose relative_to="${prefix}base_rod">0 0 ${rod_length}   0 ${pi/2} 0</pose>
+        <axis>
+          <xyz>0 1 0</xyz>
+        </axis>
       </joint>
-      <joint name="${prefix}joint_2_3" type="revolute">
-        <origin xyz="0 0 ${rod_length}" rpy="0 ${pi/2} 0"/>
-        <parent link="${prefix}rod" />
-        <child link="${prefix}external_crank" />
-        <axis xyz="0 1 0" />
-        <limit lower="${-pi}" upper="${pi}" velocity="2.0" effort="10" />
-        <mimic joint="${prefix}finger_joint" multiplier="1" offset="0" />
-      </joint>
-        <joint name="${prefix}joint_3_4" type="revolute">
-          <origin xyz="0 0 ${crank_length}" rpy="0 ${pi/2} 0"/>
-          <parent link="${prefix}external_crank" />
-          <child link="${prefix}base_rod" />
-          <axis xyz="0 1 0" />
-          <limit lower="${-pi}" upper="${pi}" velocity="2.0" effort="10" />
-          <mimic joint="${prefix}finger_joint" multiplier="-1" offset="0" />
-        </joint>
-        <link name="${prefix}tip"/>
-        <joint name="${prefix}tip_joint" type="fixed">
-          <origin xyz="${-0.5*link_width} 0 ${phalanx_length}" rpy="0 0 0"/>
-          <parent link="${prefix}phalanx" />
-          <child link="${prefix}tip" />
-        </joint>
-      <gazebo>
-        <joint name="${prefix}joint_4_1" type="revolute">
-         <parent>${prefix}base_rod</parent>
-         <child>${prefix}crank</child>
-         <pose relative_to="${prefix}base_rod">0 0 ${rod_length}   0 ${pi/2} 0</pose>
-         <axis>
-           <xyz>0 1 0</xyz>
-         </axis>
-       </joint>
-       <joint name="${prefix}joint_0_4" type="revolute">
+      <joint name="${prefix}joint_0_4" type="revolute">
         <parent>${base_name}</parent>
         <child>${prefix}base_rod</child>
@@ -97,12 +98,12 @@
         </axis>
       </joint>
-      </gazebo>
-      <gazebo reference="${prefix}phalanx">
-        <self_collide>1</self_collide>
-        <kp>100000</kp>
-        <kd>200</kd>
-        <mu1>2</mu1>
-        <mu2>2</mu2>
-      </gazebo>
+    </gazebo>
+    <gazebo reference="${prefix}phalanx">
+      <self_collide>1</self_collide>
+      <kp>100000</kp>
+      <kd>200</kd>
+      <mu1>2</mu1>
+      <mu2>2</mu2>
+    </gazebo> -->
     </xacro:macro>
 </robot>

File: urdf/gripper.xacro (robot description, xacro)
@@ -25,6 +25,6 @@
 SOFTWARE, EVEN IF ADVISED OF THE POSSIBILITY OF SUCH DAMAGE.
 -->
-<robot xmlns:xacro="http://ros.org/wiki/xacro">
-  <xacro:macro name="gripper" params="prefix">
+<robot name="parallel_gripper" xmlns:xacro="http://ros.org/wiki/xacro">
+  <xacro:macro name="gripper" params="prefix:=''">
   <xacro:include filename="$(find parallel_2f_gripper)/urdf/box.xacro" />
   <xacro:include filename="$(find parallel_2f_gripper)/urdf/finger.xacro" />
@@ -37,6 +37,39 @@
   <xacro:property name="phalanx_length" value="0.05" />
   <xacro:property name="rod_length" value="0.05" />
-  <xacro:box name="gripper_base" width="${base_x}" height="${link_height}" length="${base_z}"/>
-  <link name="${prefix}open_tip"/>
+  <xacro:box name="${prefix}gripper_base" width="${base_x}" height="${link_height}" length="${base_z}"/>
+  <!-- <link name="${prefix}fingers_link">
+    <inertial>
+      <origin xyz="0 0 0" rpy="0 0 0" />
+      <mass value="1" />
+      <inertia ixx="0.1" ixy="0.0" ixz="0.0" iyy="0.1" iyz="0.0" izz="0.1" />
+    </inertial>
+    <visual>
+      <origin xyz="0 0 ${0.5*crank_length/2}" rpy="0 0 0" />
+      <geometry>
+        <box size="${link_width} ${link_height} ${crank_length/2}"/>
+      </geometry>
+      <material name="aluminium">
+        <color rgba="${132/256} ${135/256} ${137/256} 1" />
+      </material>
+    </visual>
+    <collision>
+      <origin xyz="0 0 ${0.5*crank_length/2}" rpy="0 0 0" />
+      <geometry>
+        <box size="${link_width} ${link_height} ${crank_length/2}"/>
+      </geometry>
+      <material name="aluminium">
+        <color rgba="${132/256} ${135/256} ${137/256} 1" />
+      </material>
+    </collision>
+  </link>
+  <joint name="${prefix}fingers_joint" type="revolute">
+    <origin xyz="0 0 0.01" rpy="0 0 0"/>
+    <parent link="${prefix}gripper_base" />
+    <child link="${prefix}fingers_link" />
+    <axis xyz="0 1 0" />
+    <limit lower="${-asin(0.5*base_x/crank_length)}" upper="${1}" velocity="5.0" effort="5" />
+  </joint> -->
+<!-- Add if to include these link only for rviz  -->
+  <!-- <link name="${prefix}open_tip"/>
   <joint name="${prefix}open_tip_joint" type="fixed">
     <origin xyz="0 0 ${cos(1)*crank_length+base_z+phalanx_length}" rpy="0 0 0"/>
@@ -50,10 +83,10 @@
     <child link="${prefix}closed_tip" />
   </joint>
-    <link name="${prefix}zero_pos_tip"/>
-    <joint name="${prefix}zero_pos_tip_joint" type="fixed">
-      <origin xyz="0 0 ${crank_length+base_z+phalanx_length}" rpy="0 0 0"/>
-      <parent link="${prefix}gripper_base" />
-      <child link="${prefix}zero_pos_tip" />
-    </joint>
+  <link name="${prefix}zero_pos_tip"/>
+  <joint name="${prefix}zero_pos_tip_joint" type="fixed">
+    <origin xyz="0 0 ${crank_length+base_z+phalanx_length}" rpy="0 0 0"/>
+    <parent link="${prefix}gripper_base" />
+    <child link="${prefix}zero_pos_tip" />
+  </joint> -->
   <xacro:finger
     prefix        ="${prefix}right_"
@@ -69,4 +102,5 @@
     rot_z         ="0"
   />
+  <!-- mimic_joint   ="${prefix}fingers_joint" -->
   <xacro:finger
     prefix        ="${prefix}left_"
@@ -79,9 +113,155 @@
     base_x        ="${base_x}"
     base_z        ="${base_z}"
-    mimic_joint   =""
+    mimic_joint   ="${prefix}right_finger_joint"
     rot_z         ="${pi}"
   />
+  <!-- <link name="${prefix}central_link_1">
+    <inertial>
+      <origin xyz="0 0 0" rpy="0 0 0" />
+      <mass value="0.01" />
+      <inertia
+        ixx="0.00001"
+        ixy="0.00000"
+        ixz="0.00000"
+        iyy="0.00001"
+        iyz="0.00000"
+        izz="0.00000" />
+    </inertial>
+    <visual>
+      <origin xyz="0 0 0" rpy="0 0 0" />
+      <geometry>
+        <box size="0.001 0.09 0.001" />
+      </geometry>
+      <material name="Cyan">
+        <color rgba="0 1.0 1.0 1.0"/>
+      </material>
+    </visual>
+  </link>
+  <link name="${prefix}central_link_2">
+    <inertial>
+      <origin xyz="0 0 0" rpy="0 0 0" />
+      <mass value="0.01" />
+      <inertia
+        ixx="0.00001"
+        ixy="0.00000"
+        ixz="0.00000"
+        iyy="0.00001"
+        iyz="0.00000"
+        izz="0.00000" />
+    </inertial>
+    <visual>
+      <origin xyz="0 0 0" rpy="0 0 0" />
+      <geometry>
+        <box size="0.001 0.09 0.001" />
+      </geometry>
+      <material name="Cyan">
+        <color rgba="0 1.0 1.0 1.0"/>
+      </material>
+    </visual>
+  </link>
+  <link name="${prefix}left_link">
+    <inertial>
+      <origin xyz="0 0 0" rpy="0 0 0" />
+      <mass value="0.01" />
+      <inertia
+        ixx="0.00001"
+        ixy="0.00000"
+        ixz="0.00000"
+        iyy="0.00001"
+        iyz="0.00000"
+        izz="0.00000" />
+    </inertial>
+    <visual>
+      <origin xyz="0.075 0 0" rpy="0 0 0" />
+      <geometry>
+        <box size="0.150 0.001 0.001" />
+      </geometry>
+      <material name="Cyan">
+        <color rgba="0 1.0 1.0 1.0"/>
+      </material>
+    </visual>
+  </link>
+  <link name="${prefix}right_link">
+    <inertial>
+      <origin xyz="0 0 0" rpy="0 0 0" />
+      <mass value="0.01" />
+      <inertia
+        ixx="0.00001"
+        ixy="0.00000"
+        ixz="0.00000"
+        iyy="0.00001"
+        iyz="0.00000"
+        izz="0.00000" />
+    </inertial>
+    <visual>
+      <origin xyz="0.075 0 0" rpy="0 0 0" />
+      <geometry>
+        <box size="0.150 0.001 0.001" />
+      </geometry>
+      <material name="Cyan">
+        <color rgba="0 1.0 1.0 1.0"/>
+      </material>
+    </visual>
+  </link>
+  <joint name="${prefix}left_joint" type="continuous">
+    <origin xyz="0 0 0" rpy="0 0 0"/>
+    <parent link="${prefix}left_rod" />
+    <child link="${prefix}left_link" />
+    <axis xyz="0 1 0" />
+  </joint>
+  <joint name="${prefix}right_joint" type="continuous">
+    <origin xyz="0 0 0" rpy="0 0 0"/>
+    <parent link="${prefix}right_crank" />
+    <child link="${prefix}right_link" />
+    <axis xyz="0 1 0" />
+  </joint>
+  <joint name="${prefix}central_joint_1" type="continuous">
+    <origin xyz="0.120 0 -0.055" rpy="0 0 0"/>
+    <parent link="${prefix}right_link" />
+    <child link="${prefix}central_link_1" />
+    <axis xyz="0 1 0" />
+  </joint>
+  <joint name="${prefix}central_joint_2" type="continuous">
+    <origin xyz="0.120 0 -0.055" rpy="${pi} 0 0"/>
+    <parent link="${prefix}left_link" />
+    <child link="${prefix}central_link_2" />
+    <axis xyz="0 1 0" />
+  </joint> -->
+  <!-- <gazebo>
+    <joint name="${prefix}central_joint" type="fixed">
+      <parent>${prefix}central_link_1</parent>
+      <child>${prefix}central_link_2</child>
+      <pose relative_to="${prefix}central_link_1"> 0, 0, 0, 0, 0, 0</pose>
+      <axis>
+        <xyz expressed_in="central_link">0 1 0</xyz>
+      </axis>
+    </joint>
+    <joint name="${prefix}linear_joint_1" type="prismatic">
+      <parent>${prefix}gripper_base</parent>
+      <child>${prefix}central_link_1</child>
+      <pose relative_to="${prefix}gripper_base"> 0, 0, 0, 0, ${pi/2}, 0</pose>
+      <axis>
+        <xyz expressed_in="central_link_1">1 0 0</xyz>
+      </axis>
+    </joint>
+    <joint name="${prefix}linear_joint_2" type="prismatic">
+      <parent>${prefix}gripper_base</parent>
+      <child>${prefix}central_link_2</child>
+      <pose relative_to="${prefix}gripper_base"> 0, 0, 0, 0, ${pi/2}, 0</pose>
+      <axis>
+        <xyz expressed_in="central_link_2">1 0 0</xyz>
+      </axis>
+    </joint>
+  </gazebo> -->
+  <!-- <link name="${prefix}central_link_virtual"/>
+  <joint name="${prefix}linear_joint_virtuale_1" type="prismatic">
+    <origin xyz="0 0 0" rpy="0 ${pi/2} 0"/>
+    <parent link="${prefix}gripper_base" />
+    <child link="${prefix}central_link_virtual" />
+    <axis xyz="1 0 0" />
+    <limit lower="${-pi}" upper="${pi}" velocity="2.0" effort="10" />
+  </joint> -->
   <xacro:transmission prefix="${prefix}right_"/>
-  <xacro:transmission prefix="${prefix}left_"/>
+  <!-- <xacro:transmission prefix="${prefix}left_"/> -->
   </xacro:macro>
 </robot>

File: urdf/gripper_pybullet.xacro (robot description, xacro)
@@ -1,3 +1,3 @@
-<?xml version="1.0"?>
+<?xml version="1.0" ?>
 <!--
 Copyright (c) 2022, JRL-CARI CNR-STIIMA/UNIBS
@@ -25,7 +25,12 @@
 SOFTWARE, EVEN IF ADVISED OF THE POSSIBILITY OF SUCH DAMAGE.
 -->
-<launch>
-  <arg name="fixed" default="True" />
-  <param name="robot_description" if="$(arg fixed)" command="$(find xacro)/xacro --inorder $(find parallel_2f_gripper)/urdf/gripper_standalone.xacro" />
-  <param name="robot_description" unless="$(arg fixed)" command="$(find xacro)/xacro --inorder $(find parallel_2f_gripper)/urdf/gripper_standalone_not_fixed.xacro" />
-</launch>
+<robot name="parallel_gripper" xmlns:xacro="http://ros.org/wiki/xacro">
+  <xacro:include filename="$(find parallel_2f_gripper)/urdf/gripper.xacro" />
+  <xacro:gripper prefix=""/>
+  <gazebo>
+    <plugin name="gazebo_ros_control" filename="libgazebo_ros_control.so">
+      <robotNamespace>/gripper</robotNamespace>
+      <robotSimType>gazebo_ros_control/DefaultRobotHWSim</robotSimType>
+    </plugin>
+  </gazebo>
+</robot>

File: urdf/gripper_rviz.xacro (robot description, xacro)
@@ -25,19 +25,18 @@
 SOFTWARE, EVEN IF ADVISED OF THE POSSIBILITY OF SUCH DAMAGE.
 -->
-<launch>
-  <arg name="gui" default="True" />
-  <arg name="simulation" default="True" />
-  <param name="use_gui" value="$(arg gui)"/>
-  <include file="$(find parallel_2f_gripper)/launch/upload.launch"/>
-  <node if = "$(arg simulation)" name="joint_state_publisher" pkg="joint_state_publisher" type="joint_state_publisher">
-    <param name="/use_gui" value="false"/>
-    <param name="rate" value="500"/>
-    <rosparam param="/source_list">[/parallel_gripper/joint_states]</rosparam>
-  </node>
-  <node name="joint_target_publisher" pkg="joint_state_publisher_gui" type="joint_state_publisher_gui" >
-    <param name="rate" value="500"/>
-    <remap if = "$(arg simulation)" from="joint_states" to="/parallel_gripper/joint_target"/>
-  </node>
-  <node name="robot_state_publisher" pkg="robot_state_publisher" type="robot_state_publisher" />
-  <node name="rviz" pkg="rviz" type="rviz" args="-d $(find parallel_2f_gripper)/launch/config.rviz" required="true" />
-</launch>
+<robot name="parallel_gripper" xmlns:xacro="http://ros.org/wiki/xacro">
+  <xacro:include filename="$(find parallel_2f_gripper)/urdf/gripper.xacro" />
+  <xacro:gripper prefix=""/>
+  <link name="world"/>
+  <joint name="world_joint" type="fixed">
+    <origin xyz="0 0 0.05" rpy="${pi*0.5} 0 0"/>
+    <parent link="world" />
+    <child link="gripper_base" />
+  </joint>
+  <gazebo>
+    <plugin name="gazebo_ros_control" filename="libgazebo_ros_control.so">
+      <robotNamespace>/gripper</robotNamespace>
+      <robotSimType>gazebo_ros_control/DefaultRobotHWSim</robotSimType>
+    </plugin>
+  </gazebo>
+</robot>
