Commit message: robot_name and prefix parametrization added

File: urdf/gripper_pybullet.xacro (robot description, xacro)
@@ -25,7 +25,12 @@
 SOFTWARE, EVEN IF ADVISED OF THE POSSIBILITY OF SUCH DAMAGE.
 -->
-<robot name="parallel_gripper" xmlns:xacro="http://ros.org/wiki/xacro">
+<!-- It is required to pass the args: robot_name-->
+<robot name="$(arg robot_name)" xmlns:xacro="http://ros.org/wiki/xacro">
   <xacro:include filename="$(find parallel_2f_gripper)/urdf/gripper.xacro" />
-  <xacro:property name="prefix" value="''" />
+  <xacro:arg name="prefix" default="null"/>
+  <xacro:property name="prefix" value="'$(arg prefix)'" />
+  <xacro:if value="${prefix == 'null'}">
+    <xacro:property name="prefix" value="''" />
+  </xacro:if>
   <xacro:property name="type"   value="'pybullet'" />
   <xacro:gripper prefix="${prefix}" type="${type}"/>

File: urdf/gripper_rviz.xacro (robot description, xacro)
@@ -25,7 +25,12 @@
 SOFTWARE, EVEN IF ADVISED OF THE POSSIBILITY OF SUCH DAMAGE.
 -->
-<robot name="parallel_gripper" xmlns:xacro="http://ros.org/wiki/xacro">
+<!-- It is required to pass the args: robot_name-->
+<robot name="$(arg robot_name)" xmlns:xacro="http://ros.org/wiki/xacro">
   <xacro:include filename="$(find parallel_2f_gripper)/urdf/gripper.xacro" />
-  <xacro:property name="prefix" value="''" />
+  <xacro:arg name="prefix" default="null"/>
+  <xacro:property name="prefix" value="'$(arg prefix)'" />
+  <xacro:if value="${prefix == 'null'}">
+    <xacro:property name="prefix" value="''" />
+  </xacro:if>
   <xacro:property name="type"   value="'rviz'" />
   <xacro:gripper prefix="${prefix}" type="${type}"/>
@@ -34,5 +39,5 @@
     <origin xyz="0 0 0.05" rpy="${pi*0.5} 0 0"/>
     <parent link="world" />
-    <child link="gripper_base" />
+    <child link="${prefix}gripper_base" />
   </joint>
 </robot>
