Commit message: little changes

File: urdf/gripper_pybullet.urdf (robot description, URDF)
Before this commit: robot parallel_gripper, 11 links, 10 joints
Links:
- removed link kr_50_gripper_base
- removed link kr_50_left_base_rod
- removed link kr_50_left_crank
- removed link kr_50_left_external_crank
- removed link kr_50_left_phalanx
- removed link kr_50_left_rod
- removed link kr_50_right_base_rod
- removed link kr_50_right_crank
- removed link kr_50_right_external_crank
- removed link kr_50_right_phalanx
- removed link kr_50_right_rod
- added link gripper_base, mass 0.2; collision box size=0.1 0.05 0.05; visual box size=0.1 0.05 0.05
- added link left_base_rod, mass 0.2; collision box size=0.01 0.05 0.05; visual box size=0.01 0.05 0.05
- added link left_crank, mass 0.2; collision box size=0.01 0.05 0.07; visual box size=0.01 0.05 0.07
- added link left_external_crank, mass 0.2; collision box size=0.01 0.05 0.07; visual box size=0.01 0.05 0.07
- added link left_phalanx, mass 0.2; collision box size=0.01 0.05 0.05; visual box size=0.01 0.05 0.05
- added link left_rod, mass 0.2; collision box size=0.01 0.05 0.05; visual box size=0.01 0.05 0.05
- added link right_base_rod, mass 0.2; collision box size=0.01 0.05 0.05; visual box size=0.01 0.05 0.05
- added link right_crank, mass 0.2; collision box size=0.01 0.05 0.07; visual box size=0.01 0.05 0.07
- added link right_external_crank, mass 0.2; collision box size=0.01 0.05 0.07; visual box size=0.01 0.05 0.07
- added link right_phalanx, mass 0.2; collision box size=0.01 0.05 0.05; visual box size=0.01 0.05 0.05
- added link right_rod, mass 0.2; collision box size=0.01 0.05 0.05; visual box size=0.01 0.05 0.05
Joints:
- removed joint kr_50_left_finger_joint
- removed joint kr_50_left_joint_1_2
- removed joint kr_50_left_joint_2_3
- removed joint kr_50_left_joint_2_5
- removed joint kr_50_left_joint_3_4
- removed joint kr_50_right_finger_joint
- removed joint kr_50_right_joint_1_2
- removed joint kr_50_right_joint_2_3
- removed joint kr_50_right_joint_2_5
- removed joint kr_50_right_joint_3_4
- added joint left_finger_joint: type revolute, parent gripper_base, child left_crank, origin xyz=-0.055 0 0.05 rpy=0 0 3.141592653589793, axis 0 1 0, limit lower=-0.7956029534845354 upper=1 effort=5 velocity=5.0, mimic joint=right_finger_joint multiplier=1 offset=0
- added joint left_joint_1_2: type revolute, parent left_crank, child left_rod, origin xyz=0 0 0.07 rpy=0 1.5707963267948966 0, axis 0 1 0, limit lower=-3.141592653589793 upper=3.141592653589793 effort=10 velocity=2.0, mimic joint=left_finger_joint multiplier=-1 offset=0
- added joint left_joint_2_3: type revolute, parent left_rod, child left_external_crank, origin xyz=0 0 0.05 rpy=0 1.5707963267948966 0, axis 0 1 0, limit lower=-3.141592653589793 upper=3.141592653589793 effort=10 velocity=2.0, mimic joint=left_finger_joint multiplier=1 offset=0
- added joint left_joint_2_5: type fixed, parent left_rod, child left_phalanx, origin xyz=0 0 0 rpy=0 -1.5707963267948966 0, axis 0 1 0
- added joint left_joint_3_4: type revolute, parent left_external_crank, child left_base_rod, origin xyz=0 0 0.07 rpy=0 1.5707963267948966 0, axis 0 1 0, limit lower=-3.141592653589793 upper=3.141592653589793 effort=10 velocity=2.0, mimic joint=left_finger_joint multiplier=-1 offset=0
- added joint right_finger_joint: type revolute, parent gripper_base, child right_crank, origin xyz=0.055 0 0.05 rpy=0 0 0, axis 0 1 0, limit lower=-0.7956029534845354 upper=1 effort=5 velocity=5.0
- added joint right_joint_1_2: type revolute, parent right_crank, child right_rod, origin xyz=0 0 0.07 rpy=0 1.5707963267948966 0, axis 0 1 0, limit lower=-3.141592653589793 upper=3.141592653589793 effort=10 velocity=2.0, mimic joint=right_finger_joint multiplier=-1 offset=0
- added joint right_joint_2_3: type revolute, parent right_rod, child right_external_crank, origin xyz=0 0 0.05 rpy=0 1.5707963267948966 0, axis 0 1 0, limit lower=-3.141592653589793 upper=3.141592653589793 effort=10 velocity=2.0, mimic joint=right_finger_joint multiplier=1 offset=0
- added joint right_joint_2_5: type fixed, parent right_rod, child right_phalanx, origin xyz=0 0 0 rpy=0 -1.5707963267948966 0, axis 0 1 0
- added joint right_joint_3_4: type revolute, parent right_external_crank, child right_base_rod, origin xyz=0 0 0.07 rpy=0 1.5707963267948966 0, axis 0 1 0, limit lower=-3.141592653589793 upper=3.141592653589793 effort=10 velocity=2.0, mimic joint=right_finger_joint multiplier=-1 offset=0
