Commit message: without gearbox

File: urdf/gripper.xacro (robot description, xacro)
@@ -79,27 +79,9 @@
     base_x        ="${base_x}"
     base_z        ="${base_z}"
-    mimic_joint   ="right_finger_joint"
+    mimic_joint   =""
     rot_z         ="${pi}"
   />
-  <gazebo>
-    <!-- gearbox between the two finger (like mimic for URDF) -->
-    <joint name="${prefix}left_right" type="gearbox">
-     <parent>${prefix}right_crank</parent>
-     <child>${prefix}left_crank</child>
-     <!-- movements are computed between:
-     - parent and gearbox_reference_body
-     - child and gearbox_reference_body
-     -->
-     <gearbox_reference_body>${prefix}gripper_base</gearbox_reference_body>
-     <!-- the movement has already a negative sign -->
-     <gearbox_ratio>1</gearbox_ratio>
-     <!-- pose does not care -->
-     <pose relative_to="gripper_base">0 0 0 0 0 0</pose>
-     <axis>
-       <xyz>0 1 0</xyz>
-     </axis>
-   </joint>
-  </gazebo>
   <xacro:transmission prefix="${prefix}right_"/>
+  <xacro:transmission prefix="${prefix}left_"/>
   </xacro:macro>
 </robot>

File: urdf/gripper_standalone_not_fixed.xacro (robot description, xacro)
@@ -1,3 +1,3 @@
-<?xml version="1.0"?>
+<?xml version="1.0" ?>
 <!--
 Copyright (c) 2022, JRL-CARI CNR-STIIMA/UNIBS
@@ -25,7 +25,12 @@
 SOFTWARE, EVEN IF ADVISED OF THE POSSIBILITY OF SUCH DAMAGE.
 -->
-<launch>
-  <arg name="fixed" default="True" />
-  <param name="robot_description" if="$(arg fixed)" command="$(find xacro)/xacro --inorder $(find parallel_2f_gripper)/urdf/gripper_standalone.xacro" />
-  <param name="robot_description" unless="$(arg fixed)" command="$(find xacro)/xacro --inorder $(find parallel_2f_gripper)/urdf/gripper_standalone_not_fixed.xacro" />
-</launch>
+<robot name="gripper" xmlns:xacro="http://ros.org/wiki/xacro">
+  <xacro:include filename="$(find parallel_2f_gripper)/urdf/gripper.xacro" />
+  <xacro:gripper prefix=""/>
+  <gazebo>
+    <plugin name="gazebo_ros_control" filename="libgazebo_ros_control.so">
+      <robotNamespace>/gripper</robotNamespace>
+      <robotSimType>gazebo_ros_control/DefaultRobotHWSim</robotSimType>
+    </plugin>
+  </gazebo>
+</robot>

Commit message: ready for test

File: urdf/gripper.xacro (robot description, xacro)
@@ -26,5 +26,5 @@
 -->
 <robot name="parallel_gripper" xmlns:xacro="http://ros.org/wiki/xacro">
-  <xacro:macro name="gripper" params="prefix:=''">
+<xacro:macro name="gripper" params="prefix:='' type:=rviz">
   <xacro:include filename="$(find parallel_2f_gripper)/urdf/box.xacro" />
   <xacro:include filename="$(find parallel_2f_gripper)/urdf/finger.xacro" />
@@ -38,55 +38,24 @@
   <xacro:property name="rod_length" value="0.05" />
   <xacro:box name="${prefix}gripper_base" width="${base_x}" height="${link_height}" length="${base_z}"/>
-  <!-- <link name="${prefix}fingers_link">
-    <inertial>
-      <origin xyz="0 0 0" rpy="0 0 0" />
-      <mass value="1" />
-      <inertia ixx="0.1" ixy="0.0" ixz="0.0" iyy="0.1" iyz="0.0" izz="0.1" />
-    </inertial>
-    <visual>
-      <origin xyz="0 0 ${0.5*crank_length/2}" rpy="0 0 0" />
-      <geometry>
-        <box size="${link_width} ${link_height} ${crank_length/2}"/>
-      </geometry>
-      <material name="aluminium">
-        <color rgba="${132/256} ${135/256} ${137/256} 1" />
-      </material>
-    </visual>
-    <collision>
-      <origin xyz="0 0 ${0.5*crank_length/2}" rpy="0 0 0" />
-      <geometry>
-        <box size="${link_width} ${link_height} ${crank_length/2}"/>
-      </geometry>
-      <material name="aluminium">
-        <color rgba="${132/256} ${135/256} ${137/256} 1" />
-      </material>
-    </collision>
-  </link>
-  <joint name="${prefix}fingers_joint" type="revolute">
-    <origin xyz="0 0 0.01" rpy="0 0 0"/>
-    <parent link="${prefix}gripper_base" />
-    <child link="${prefix}fingers_link" />
-    <axis xyz="0 1 0" />
-    <limit lower="${-asin(0.5*base_x/crank_length)}" upper="${1}" velocity="5.0" effort="5" />
-  </joint> -->
-<!-- Add if to include these link only for rviz  -->
-  <!-- <link name="${prefix}open_tip"/>
-  <joint name="${prefix}open_tip_joint" type="fixed">
-    <origin xyz="0 0 ${cos(1)*crank_length+base_z+phalanx_length}" rpy="0 0 0"/>
-    <parent link="${prefix}gripper_base" />
-    <child link="${prefix}open_tip" />
-  </joint>
-  <link name="${prefix}closed_tip"/>
-  <joint name="${prefix}closed_tip_joint" type="fixed">
-    <origin xyz="0 0 ${cos(asin(0.5*base_x/crank_length))*crank_length+base_z+phalanx_length}" rpy="0 0 0"/>
-    <parent link="${prefix}gripper_base" />
-    <child link="${prefix}closed_tip" />
-  </joint>
-  <link name="${prefix}zero_pos_tip"/>
-  <joint name="${prefix}zero_pos_tip_joint" type="fixed">
-    <origin xyz="0 0 ${crank_length+base_z+phalanx_length}" rpy="0 0 0"/>
-    <parent link="${prefix}gripper_base" />
-    <child link="${prefix}zero_pos_tip" />
-  </joint> -->
+  <xacro:if value="${type == 'rviz'}">
+    <link name="${prefix}open_tip"/>
+    <joint name="${prefix}open_tip_joint" type="fixed">
+      <origin xyz="0 0 ${cos(1)*crank_length+base_z+phalanx_length}" rpy="0 0 0"/>
+      <parent link="${prefix}gripper_base" />
+      <child link="${prefix}open_tip" />
+    </joint>
+    <link name="${prefix}closed_tip"/>
+    <joint name="${prefix}closed_tip_joint" type="fixed">
+      <origin xyz="0 0 ${cos(asin(0.5*base_x/crank_length))*crank_length+base_z+phalanx_length}" rpy="0 0 0"/>
+      <parent link="${prefix}gripper_base" />
+      <child link="${prefix}closed_tip" />
+    </joint>
+    <link name="${prefix}zero_pos_tip"/>
+    <joint name="${prefix}zero_pos_tip_joint" type="fixed">
+      <origin xyz="0 0 ${crank_length+base_z+phalanx_length}" rpy="0 0 0"/>
+      <parent link="${prefix}gripper_base" />
+      <child link="${prefix}zero_pos_tip" />
+    </joint>
+  </xacro:if>
   <xacro:finger
     prefix        ="${prefix}right_"
@@ -102,5 +71,4 @@
     rot_z         ="0"
   />
-  <!-- mimic_joint   ="${prefix}fingers_joint" -->
   <xacro:finger
     prefix        ="${prefix}left_"
@@ -116,152 +84,6 @@
     rot_z         ="${pi}"
   />
-  <!-- <link name="${prefix}central_link_1">
-    <inertial>
-      <origin xyz="0 0 0" rpy="0 0 0" />
-      <mass value="0.01" />
-      <inertia
-        ixx="0.00001"
-        ixy="0.00000"
-        ixz="0.00000"
-        iyy="0.00001"
-        iyz="0.00000"
-        izz="0.00000" />
-    </inertial>
-    <visual>
-      <origin xyz="0 0 0" rpy="0 0 0" />
-      <geometry>
-        <box size="0.001 0.09 0.001" />
-      </geometry>
-      <material name="Cyan">
-        <color rgba="0 1.0 1.0 1.0"/>
-      </material>
-    </visual>
-  </link>
-  <link name="${prefix}central_link_2">
-    <inertial>
-      <origin xyz="0 0 0" rpy="0 0 0" />
-      <mass value="0.01" />
-      <inertia
-        ixx="0.00001"
-        ixy="0.00000"
-        ixz="0.00000"
-        iyy="0.00001"
-        iyz="0.00000"
-        izz="0.00000" />
-    </inertial>
-    <visual>
-      <origin xyz="0 0 0" rpy="0 0 0" />
-      <geometry>
-        <box size="0.001 0.09 0.001" />
-      </geometry>
-      <material name="Cyan">
-        <color rgba="0 1.0 1.0 1.0"/>
-      </material>
-    </visual>
-  </link>
-  <link name="${prefix}left_link">
-    <inertial>
-      <origin xyz="0 0 0" rpy="0 0 0" />
-      <mass value="0.01" />
-      <inertia
-        ixx="0.00001"
-        ixy="0.00000"
-        ixz="0.00000"
-        iyy="0.00001"
-        iyz="0.00000"
-        izz="0.00000" />
-    </inertial>
-    <visual>
-      <origin xyz="0.075 0 0" rpy="0 0 0" />
-      <geometry>
-        <box size="0.150 0.001 0.001" />
-      </geometry>
-      <material name="Cyan">
-        <color rgba="0 1.0 1.0 1.0"/>
-      </material>
-    </visual>
-  </link>
-  <link name="${prefix}right_link">
-    <inertial>
-      <origin xyz="0 0 0" rpy="0 0 0" />
-      <mass value="0.01" />
-      <inertia
-        ixx="0.00001"
-        ixy="0.00000"
-        ixz="0.00000"
-        iyy="0.00001"
-        iyz="0.00000"
-        izz="0.00000" />
-    </inertial>
-    <visual>
-      <origin xyz="0.075 0 0" rpy="0 0 0" />
-      <geometry>
-        <box size="0.150 0.001 0.001" />
-      </geometry>
-      <material name="Cyan">
-        <color rgba="0 1.0 1.0 1.0"/>
-      </material>
-    </visual>
-  </link>
-  <joint name="${prefix}left_joint" type="continuous">
-    <origin xyz="0 0 0" rpy="0 0 0"/>
-    <parent link="${prefix}left_rod" />
-    <child link="${prefix}left_link" />
-    <axis xyz="0 1 0" />
-  </joint>
-  <joint name="${prefix}right_joint" type="continuous">
-    <origin xyz="0 0 0" rpy="0 0 0"/>
-    <parent link="${prefix}right_crank" />
-    <child link="${prefix}right_link" />
-    <axis xyz="0 1 0" />
-  </joint>
-  <joint name="${prefix}central_joint_1" type="continuous">
-    <origin xyz="0.120 0 -0.055" rpy="0 0 0"/>
-    <parent link="${prefix}right_link" />
-    <child link="${prefix}central_link_1" />
-    <axis xyz="0 1 0" />
-  </joint>
-  <joint name="${prefix}central_joint_2" type="continuous">
-    <origin xyz="0.120 0 -0.055" rpy="${pi} 0 0"/>
-    <parent link="${prefix}left_link" />
-    <child link="${prefix}central_link_2" />
-    <axis xyz="0 1 0" />
-  </joint> -->
-  <!-- <gazebo>
-    <joint name="${prefix}central_joint" type="fixed">
-      <parent>${prefix}central_link_1</parent>
-      <child>${prefix}central_link_2</child>
-      <pose relative_to="${prefix}central_link_1"> 0, 0, 0, 0, 0, 0</pose>
-      <axis>
-        <xyz expressed_in="central_link">0 1 0</xyz>
-      </axis>
-    </joint>
-    <joint name="${prefix}linear_joint_1" type="prismatic">
-      <parent>${prefix}gripper_base</parent>
-      <child>${prefix}central_link_1</child>
-      <pose relative_to="${prefix}gripper_base"> 0, 0, 0, 0, ${pi/2}, 0</pose>
-      <axis>
-        <xyz expressed_in="central_link_1">1 0 0</xyz>
-      </axis>
-    </joint>
-    <joint name="${prefix}linear_joint_2" type="prismatic">
-      <parent>${prefix}gripper_base</parent>
-      <child>${prefix}central_link_2</child>
-      <pose relative_to="${prefix}gripper_base"> 0, 0, 0, 0, ${pi/2}, 0</pose>
-      <axis>
-        <xyz expressed_in="central_link_2">1 0 0</xyz>
-      </axis>
-    </joint>
-  </gazebo> -->
-  <!-- <link name="${prefix}central_link_virtual"/>
-  <joint name="${prefix}linear_joint_virtuale_1" type="prismatic">
-    <origin xyz="0 0 0" rpy="0 ${pi/2} 0"/>
-    <parent link="${prefix}gripper_base" />
-    <child link="${prefix}central_link_virtual" />
-    <axis xyz="1 0 0" />
-    <limit lower="${-pi}" upper="${pi}" velocity="2.0" effort="10" />
-  </joint> -->
   <xacro:transmission prefix="${prefix}right_"/>
-  <!-- <xacro:transmission prefix="${prefix}left_"/> -->
-  </xacro:macro>
+  <xacro:transmission prefix="${prefix}left_"/>
+</xacro:macro>
 </robot>

File: urdf/gripper_pybullet.xacro (robot description, xacro)
@@ -27,10 +27,6 @@
 <robot name="parallel_gripper" xmlns:xacro="http://ros.org/wiki/xacro">
   <xacro:include filename="$(find parallel_2f_gripper)/urdf/gripper.xacro" />
-  <xacro:gripper prefix=""/>
-  <gazebo>
-    <plugin name="gazebo_ros_control" filename="libgazebo_ros_control.so">
-      <robotNamespace>/gripper</robotNamespace>
-      <robotSimType>gazebo_ros_control/DefaultRobotHWSim</robotSimType>
-    </plugin>
-  </gazebo>
+  <xacro:property name="prefix" value="''" />
+  <xacro:property name="type"   value="'pybullet'" />
+  <xacro:gripper prefix="${prefix}" type="${type}"/>
 </robot>

File: urdf/gripper_rviz.xacro (robot description, xacro)
@@ -27,5 +27,7 @@
 <robot name="parallel_gripper" xmlns:xacro="http://ros.org/wiki/xacro">
   <xacro:include filename="$(find parallel_2f_gripper)/urdf/gripper.xacro" />
-  <xacro:gripper prefix=""/>
+  <xacro:property name="prefix" value="''" />
+  <xacro:property name="type"   value="'rviz'" />
+  <xacro:gripper prefix="${prefix}" type="${type}"/>
   <link name="world"/>
   <joint name="world_joint" type="fixed">
@@ -34,9 +36,3 @@
     <child link="gripper_base" />
   </joint>
-  <gazebo>
-    <plugin name="gazebo_ros_control" filename="libgazebo_ros_control.so">
-      <robotNamespace>/gripper</robotNamespace>
-      <robotSimType>gazebo_ros_control/DefaultRobotHWSim</robotSimType>
-    </plugin>
-  </gazebo>
 </robot>

Commit message: End first gauss

File: urdf/gripper.xacro (robot description, xacro)
@@ -25,5 +25,5 @@
 SOFTWARE, EVEN IF ADVISED OF THE POSSIBILITY OF SUCH DAMAGE.
 -->
-<robot name="parallel_gripper" xmlns:xacro="http://ros.org/wiki/xacro">
+<robot xmlns:xacro="http://ros.org/wiki/xacro">
 <xacro:macro name="gripper" params="prefix:='' type:=rviz">
   <xacro:include filename="$(find parallel_2f_gripper)/urdf/box.xacro" />

File: urdf/gripper_pybullet.urdf (robot description, URDF)
Before this commit: robot parallel_gripper, 11 links, 10 joints
Links:
- removed link gripper_base
- removed link left_base_rod
- removed link left_crank
- removed link left_external_crank
- removed link left_phalanx
- removed link left_rod
- removed link right_base_rod
- removed link right_crank
- removed link right_external_crank
- removed link right_phalanx
- removed link right_rod
- added link parallel_gripper_gripper_base, mass 0.2; collision box size=0.1 0.05 0.05; visual box size=0.1 0.05 0.05
- added link parallel_gripper_left_base_rod, mass 0.2; collision box size=0.01 0.05 0.05; visual box size=0.01 0.05 0.05
- added link parallel_gripper_left_crank, mass 0.2; collision box size=0.01 0.05 0.07; visual box size=0.01 0.05 0.07
- added link parallel_gripper_left_external_crank, mass 0.2; collision box size=0.01 0.05 0.07; visual box size=0.01 0.05 0.07
- added link parallel_gripper_left_phalanx, mass 0.2; collision box size=0.01 0.05 0.05; visual box size=0.01 0.05 0.05
- added link parallel_gripper_left_rod, mass 0.2; collision box size=0.01 0.05 0.05; visual box size=0.01 0.05 0.05
- added link parallel_gripper_right_base_rod, mass 0.2; collision box size=0.01 0.05 0.05; visual box size=0.01 0.05 0.05
- added link parallel_gripper_right_crank, mass 0.2; collision box size=0.01 0.05 0.07; visual box size=0.01 0.05 0.07
- added link parallel_gripper_right_external_crank, mass 0.2; collision box size=0.01 0.05 0.07; visual box size=0.01 0.05 0.07
- added link parallel_gripper_right_phalanx, mass 0.2; collision box size=0.01 0.05 0.05; visual box size=0.01 0.05 0.05
- added link parallel_gripper_right_rod, mass 0.2; collision box size=0.01 0.05 0.05; visual box size=0.01 0.05 0.05
Joints:
- removed joint left_finger_joint
- removed joint left_joint_1_2
- removed joint left_joint_2_3
- removed joint left_joint_2_5
- removed joint left_joint_3_4
- removed joint right_finger_joint
- removed joint right_joint_1_2
- removed joint right_joint_2_3
- removed joint right_joint_2_5
- removed joint right_joint_3_4
- added joint parallel_gripper_left_finger_joint: type revolute, parent parallel_gripper_gripper_base, child parallel_gripper_left_crank, origin xyz=-0.055 0 0.05 rpy=0 0 3.141592653589793, axis 0 1 0, limit lower=-0.7956029534845354 upper=1 effort=5 velocity=5.0, mimic joint=parallel_gripper_right_finger_joint multiplier=1 offset=0
- added joint parallel_gripper_left_joint_1_2: type revolute, parent parallel_gripper_left_crank, child parallel_gripper_left_rod, origin xyz=0 0 0.07 rpy=0 1.5707963267948966 0, axis 0 1 0, limit lower=-3.141592653589793 upper=3.141592653589793 effort=10 velocity=2.0, mimic joint=parallel_gripper_left_finger_joint multiplier=-1 offset=0
- added joint parallel_gripper_left_joint_2_3: type revolute, parent parallel_gripper_left_rod, child parallel_gripper_left_external_crank, origin xyz=0 0 0.05 rpy=0 1.5707963267948966 0, axis 0 1 0, limit lower=-3.141592653589793 upper=3.141592653589793 effort=10 velocity=2.0, mimic joint=parallel_gripper_left_finger_joint multiplier=1 offset=0
- added joint parallel_gripper_left_joint_2_5: type fixed, parent parallel_gripper_left_rod, child parallel_gripper_left_phalanx, origin xyz=0 0 0 rpy=0 -1.5707963267948966 0, axis 0 1 0
- added joint parallel_gripper_left_joint_3_4: type revolute, parent parallel_gripper_left_external_crank, child parallel_gripper_left_base_rod, origin xyz=0 0 0.07 rpy=0 1.5707963267948966 0, axis 0 1 0, limit lower=-3.141592653589793 upper=3.141592653589793 effort=10 velocity=2.0, mimic joint=parallel_gripper_left_finger_joint multiplier=-1 offset=0
- added joint parallel_gripper_right_finger_joint: type revolute, parent parallel_gripper_gripper_base, child parallel_gripper_right_crank, origin xyz=0.055 0 0.05 rpy=0 0 0, axis 0 1 0, limit lower=-0.7956029534845354 upper=1 effort=5 velocity=5.0
- added joint parallel_gripper_right_joint_1_2: type revolute, parent parallel_gripper_right_crank, child parallel_gripper_right_rod, origin xyz=0 0 0.07 rpy=0 1.5707963267948966 0, axis 0 1 0, limit lower=-3.141592653589793 upper=3.141592653589793 effort=10 velocity=2.0, mimic joint=parallel_gripper_right_finger_joint multiplier=-1 offset=0
- added joint parallel_gripper_right_joint_2_3: type revolute, parent parallel_gripper_right_rod, child parallel_gripper_right_external_crank, origin xyz=0 0 0.05 rpy=0 1.5707963267948966 0, axis 0 1 0, limit lower=-3.141592653589793 upper=3.141592653589793 effort=10 velocity=2.0, mimic joint=parallel_gripper_right_finger_joint multiplier=1 offset=0
- added joint parallel_gripper_right_joint_2_5: type fixed, parent parallel_gripper_right_rod, child parallel_gripper_right_phalanx, origin xyz=0 0 0 rpy=0 -1.5707963267948966 0, axis 0 1 0
- added joint parallel_gripper_right_joint_3_4: type revolute, parent parallel_gripper_right_external_crank, child parallel_gripper_right_base_rod, origin xyz=0 0 0.07 rpy=0 1.5707963267948966 0, axis 0 1 0, limit lower=-3.141592653589793 upper=3.141592653589793 effort=10 velocity=2.0, mimic joint=parallel_gripper_right_finger_joint multiplier=-1 offset=0

File: urdf/gripper_pybullet.xacro (robot description, xacro)
@@ -28,9 +28,6 @@
 <robot name="$(arg robot_name)" xmlns:xacro="http://ros.org/wiki/xacro">
   <xacro:include filename="$(find parallel_2f_gripper)/urdf/gripper.xacro" />
-  <xacro:arg name="prefix" default="null"/>
+  <xacro:arg name="prefix" default=""/>
   <xacro:property name="prefix" value="'$(arg prefix)'" />
-  <xacro:if value="${prefix == 'null'}">
-    <xacro:property name="prefix" value="''" />
-  </xacro:if>
   <xacro:property name="type"   value="'pybullet'" />
   <xacro:gripper prefix="${prefix}" type="${type}"/>
